File: bypass_crossmix.kicad_pcb (KiCad board)
At the start: 2 copper layers, 70 x 50 mm, 58 parts, among them K1 RELAY-HLS8L-DC5V-S-C(5P-19X15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, K2 RELAY-HLS8L-DC5V-S-C(5P-19X15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, K3 RELAY-HLS8L-DC5V-S-C(5P-19X15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, K4 RELAY-HLS8L-DC5V-S-C(5P-19X15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, P1 STATUS LED, P2 SWITCH, P3 DRYWET, P4 5V, P5 9V, P6 OUT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

Commit message: Latest changes
Parts:
- removed C21: 100n, Capacitors_SMD:C_0603_HandSoldering
- removed P4: 5V, Pin_Headers:Pin_Header_Straight_1x02
- added D2: RED, LEDs:LED-0603, F.Cu at (170.8, 109.9)
- added D3: GREEN, LEDs:LED-0603, F.Cu at (182.2, 109.9)
- added R22: 150, Resistors_SMD:R_0603_HandSoldering, F.Cu at (182.2, 106.2)
- added R23: 12, Resistors_SMD:R_0603_HandSoldering, B.Cu at (151.1, 106.0)
- added R24: 12, Resistors_SMD:R_0603_HandSoldering, F.Cu at (152.6, 97.8)
- C1, C2, C3, C4, C6, C7, C8, C9: footprint Capacitors_Elko_ThroughHole:Elko_vert_11x5mm_RM2.5_CopperClear -> Capacitors_ThroughHole:C_Radial_D5_L11_P2
- C10: value DNM -> 100u; footprint Capacitors_Elko_ThroughHole:Elko_vert_11x5mm_RM2.5_CopperClear -> Capacitors_ThroughHole:C_Radial_D5_L11_P2
- C12: moved to B.Cu
- D1: footprint Seeed-OPL-Diode:DO-214AC -> Diodes_SMD:SMA_Handsoldering
- R15: value 1 -> 180
- moved R15 16.1 mm to (170.8, 105.9), turned to 90 degrees
- moved C12 8.89 mm to (148.6, 106.0), turned to 270 degrees
- moved C9 7.88 mm to (201.7, 95.5)
- moved C8 5.97 mm to (209.8, 95.2)
- moved P1 3.81 mm to (174.0, 111.8)
- moved R1 3.81 mm to (174.0, 106.0)
- moved R2 3.81 mm to (179.7, 106.0)
- moved R5 3.34 mm to (147.8, 97.8), turned to 0 degrees
- moved R10 3.27 mm to (206.8, 98.0)
- moved C10 2.54 mm to (156.3, 95.2), turned to 90 degrees
- moved D1 0.63 mm to (179.6, 80.6)
- moved U4 0.63 mm to (150.5, 102.9)
Connections:
- C10 pad 1: Net-(C10-Pad1) -> +5V
- D1 pad 2: Net-(C10-Pad1) -> -5V
- K1 pad 3: Net-(C10-Pad1) -> Net-(K1-Pad3)
- K2 pad 3: Net-(C10-Pad1) -> Net-(K1-Pad3)
- K3 pad 2: Net-(D1-Pad1) -> Net-(K1-Pad3)
- K3 pad 3: Net-(C10-Pad1) -> -5V
- K4 pad 2: Net-(D1-Pad1) -> Net-(K1-Pad3)
- K4 pad 3: Net-(C10-Pad1) -> -5V
- P2 pad 2: VCC -> +5V
- P5 pad 2: +5V -> Net-(P5-Pad2)
- R15 pad 1: Net-(C10-Pad1) -> Net-(D2-Pad2)
- R15 pad 2: -5V -> Net-(P2-Pad1)
- U4 pad 1: GND -> Net-(R24-Pad2)
Routing:
- net Net-(C10-Pad1): track 81.2 -> 0.00 mm
- net Net-(K1-Pad3): track 0.00 -> 39.8 mm
- net +5V: track 49.0 -> 84.7 mm, vias 0 -> 2
- net VCC: track 26.5 -> 0.00 mm
- net (no net): track 0.00 -> 15.2 mm, vias 0 -> 4
- net GND: track 90.0 -> 103.8 mm, vias 3 -> 6
- net Net-(C11-Pad2): track 19.2 -> 9.91 mm
- net Net-(C13-Pad2): track 13.4 -> 22.5 mm, vias 2 -> 0
- net Net-(P2-Pad1): track 14.3 -> 22.8 mm, vias 0 -> 1
- net Net-(C7-Pad1): track 40.4 -> 34.5 mm, vias 1 -> 2
- net Net-(C16-Pad2): track 46.0 -> 40.1 mm
- net Net-(C9-Pad2): track 13.3 -> 7.45 mm
- net Net-(D1-Pad1): track 102.3 -> 97.2 mm, vias 1 -> 2
- net Net-(P5-Pad2): track 0.00 -> 4.77 mm
- net -5V: track 492.1 -> 487.4 mm, vias 51 -> 59
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Other:
- net class Power added: clearance 0.2, trace_width 0.5, via_dia 0.6, via_drill 0.4
- board text added: "COSMO MIX 1.1"
- board text removed: "5V"
- board text removed: "COSMO MIX 1.0"
