File: bypass_crossmix.sch (KiCad schematic (older format))
At the start: 58 parts, among them K1 RELAY-HLS8L-DC5V-S-C(5P-19X15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, K2 RELAY-HLS8L-DC5V-S-C(5P-19X15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, K3 RELAY-HLS8L-DC5V-S-C(5P-19X15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, K4 RELAY-HLS8L-DC5V-S-C(5P-19X15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, P1 STATUS LED, P2 SWITCH, P3 DRYWET, P4 5V, P5 9V, P6 OUT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

Commit message: Latest changes
Parts:
- removed C21: 100n, Capacitors_SMD:C_0603_HandSoldering, symbol C
- removed P4: 5V, Pin_Headers:Pin_Header_Straight_1x02, symbol CONN_01X02
- added D2: RED, LEDs:LED-0603, symbol LED
- added D3: GREEN, LEDs:LED-0603, symbol LED
- added R22: 150, Resistors_SMD:R_0603_HandSoldering, symbol R
- added R23, R24: 12, Resistors_SMD:R_0603_HandSoldering, symbol R
- C1, C2, C3, C4, C6, C7, C8, C9: footprint Capacitors_Elko_ThroughHole:Elko_vert_11x5mm_RM2.5_CopperClear -> Capacitors_ThroughHole:C_Radial_D5_L11_P2
- C10: value DNM -> 100u; footprint Capacitors_Elko_ThroughHole:Elko_vert_11x5mm_RM2.5_CopperClear -> Capacitors_ThroughHole:C_Radial_D5_L11_P2
- D1: footprint Seeed-OPL-Diode:DO-214AC -> Diodes_SMD:SMA_Handsoldering
- R15: value 1 -> 180
- U2: symbol TL074 -> TL074-RESCUE-bypass_crossmix
- U4: symbol LM358 -> LM358-RESCUE-bypass_crossmix
Connections:
- net VCC is gone; now on net +5V: P2.2 (P2)
- net +5V: now also C10.1, R23.1; no longer P5.2 (P2)
- net -5V: now also D1.2 (A), K3.3 (V-), K4.3 (V-), D2.1 (K), D3.1 (K); no longer R15.2
- net GND: now also R24.1; no longer U4.1
- net at D1.1 (K), K1.2 (V+), K2.2 (V+)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: now also R22.1; no longer K3.2 (V+), K4.2 (V+)
- net at P2.1 (P1), R1.2: now also R15.2
- new net: K1.3 (V-), K2.3 (V-), K3.2 (V+), K4.2 (V+)
- new net: R24.2, U4.1
- new net: P5.2 (P2), R23.2
- new net: D3.2 (A), R22.2
- new net: D2.2 (A), R15.1
Other:
- moved on the sheet: P5
